File: Esmeril-Placa para banca avaliadora/Esmeril espelho.kicad_pcb (KiCad board)
At the start: 2 copper layers, 108 x 85.1 mm, 27 parts, among them J1 Entrada 12V, J10 CONTATOR, J2 Display OLED 0,96, J3 MFRC522, J4 MICRO SERVO 9G, J9 BUZER, SW1 RESET, SW2 RESET, SW3 ACRILICO, SW4 INFRAVERMELHO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

Commit message: Atualização
Routing:
- net GND: track 36.8 -> 0.00 mm, vias 17 -> 15
- net SS: track 50.9 -> 43.3 mm
- net MISO: track 45.7 -> 40.6 mm
Changed lines of the file:
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@@
     (thickness 1.6)
     (drawings 4)
-    (tracks 222)
+    (tracks 211)
     (zones 0)
     (modules 27)
@@
   (via (at 142.24 133.35) (size 1.5) (drill 0.8) (layers F.Cu B.Cu) (net 1))
   (via (at 135.89 133.35) (size 1.5) (drill 0.8) (layers F.Cu B.Cu) (net 1))
-  (via (at 160.02 81.28) (size 1.5) (drill 0.8) (layers F.Cu B.Cu) (net 1))
-  (via (at 165.1 81.28) (size 1.5) (drill 0.8) (layers F.Cu B.Cu) (net 1))
-  (segment (start 160.02 81.28) (end 165.1 81.28) (width 1) (layer F.Cu) (net 1))
-  (segment (start 162.56 121.92) (end 167.64 121.92) (width 1) (layer F.Cu) (net 1))
-  (segment (start 196.85 123.19) (end 201.93 123.19) (width 1) (layer F.Cu) (net 1))
-  (segment (start 142.24 133.35) (end 135.89 133.35) (width 1) (layer F.Cu) (net 1))
-  (segment (start 121.92 121.92) (end 116.84 121.92) (width 1) (layer F.Cu) (net 1))
-  (segment (start 191.77 87.63) (end 191.77 82.55) (width 1) (layer F.Cu) (net 1))
-  (segment (start 189.23 69.85) (end 189.23 64.77) (width 1) (layer F.Cu) (net 1))
   (via (at 190.5 129.54) (size 1.5) (drill 0.8) (layers F.Cu B.Cu) (net 10))
   (via (at 182.88 129.54) (size 1.5) (drill 0.8) (layers F.Cu B.Cu) (net 10))
@@
   (segment (start 182.88 131.5) (end 179.07 135.31) (width 1) (layer B.Cu) (net 10))
   (segment (start 182.88 129.54) (end 182.88 131.5) (width 1) (layer B.Cu) (net 10))
-  (segment (start 190.5 129.54) (end 182.88 129.54) (width 1) (layer F.Cu) (net 10))
   (segment (start 181.22 103.216) (end 183.47 103.216) (width 1) (layer B.Cu) (net 11))
   (segment (start 181.61 137.16) (end 180.0596 138.7104) (width 1) (layer B.Cu) (net 11))
@@
   (segment (start 190.5 133.35) (end 186.69 137.16) (width 1) (layer B.Cu) (net 13))
   (segment (start 190.5 132.08) (end 190.5 133.35) (width 1) (layer B.Cu) (net 13))
-  (segment (start 190.5 132.08) (end 185.42 132.08) (width 1) (layer F.Cu) (net 13))
   (segment (start 134.76 77.4) (end 136.56 77.4) (width 1) (layer B.Cu) (net 16))
   (segment (start 140.97 69.85) (end 140.97 71.7) (width 1) (layer B.Cu) (net 16))
